Commit message: Merge back to jyp0802 fork

File: urdf/kobuki_2d.urdf (robot description, URDF)
Before this commit: robot hubo_3d, 3 links, 2 joints
Joints:
- joint velodyne_joint: origin xyz=0. 0. 0.99 rpy=0. 0. 0. -> xyz=0 0 0.46 rpy=0 0 0

File: urdf/kobuki_3d.urdf (robot description, URDF)
Before this commit: robot hubo_3d, 3 links, 2 joints
Joints:
- joint velodyne_joint: origin xyz=0. 0. 0.99 rpy=0. 0. 0. -> xyz=0 0 0.5 rpy=0 0 0
